File: DC.kicad_sch (KiCad schematic)
At the start: 37 parts, among them U6 MCP2551-I-P, U7 NUCLEO-F302R8

Commit message: pcb routing, reassignment of stm32 pins
Parts:
- added F6: ~, DriverControlsLib:FUSE-TH_BD5.4-W22.5-P27.5-D0.8, symbol DriverControlsLib:0001.2511.TR
Connections:
- net AccelIn: now also U7.CN10_23 (PA8); no longer U7.CN7_32 (PA4)
- net BrakeLightOut: now also U7.CN10_2 (PC8); no longer U7.CN7_3 (PC12)
- net CAN_H: now also a3.6
- net CAN_L: now also a3.5
- net DIExtra1: no longer U7.CN10_25 (PB10)
- net DIExtra2: no longer U7.CN10_22 (PB2)
- net DRLLeftOut: now also U7.CN10_6 (PC5); no longer U7.CN7_4 (PD2)
- net DRLRightOut: now also U7.CN10_16 (PB12); no longer U7.CN10_27 (PB4)
- net Drive: now also U7.CN10_26 (PA7), a3.2; no longer U7.CN10_19 (PC7), a3.1
- net GearSelector: now also a2.6; no longer a2.5
- net HazardButton: now also U7.CN7_38 (PC0), a2.5; no longer U7.CN10_23 (PA8), a2.6
- net LSignalLightButton: now also U7.CN10_25 (PB10); no longer U7.CN10_2 (PC8)
- net LSignalLightOut: now also U7.CN10_18 (PB11); no longer U7.CN7_1 (PC10)
- net Neutral: now also U7.CN10_28 (PA6), a3.3; no longer U7.CN10_15 (PB15), a3.2
- net RSignalLightButton: now also U7.CN10_24 (PB1)
- net RSignalLightOut: now also U7.CN10_4 (PC6); no longer U7.CN7_2 (PC11)
- net Reverse: now also U7.CN10_30 (PA5), a3.4; no longer U7.CN10_4 (PC6), a3.3
- net SupBattMonitor: now also U7.CN10_22 (PB2); no longer U7.CN7_38 (PC0)
- net SupBattery: now also a3.1; no longer a3.4
- net ThermalShutoff: now also U7.CN10_33 (PA10); no longer U7.CN7_17 (PA15)
- net UART_RX: now also a4.5; no longer a4.6
- net UART_TX: now also a4.6; no longer a4.5
- net VCC: now also F6.2; no longer U7.CN7_24 (VIN)
- new net: F6.1, U7.CN7_24 (VIN)
- no-connect marks 46 -> 36
Changed lines of the file:
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@@
 		)
 	)
-	(label "Reverse"
+	(label "RSignalLightOut"
 		(at 264.16 109.22 0)
 		(fields_autoplaced yes)
@@
 		)
 	)
+	(label "LSignalLightOut"
+		(at 264.16 127 0)
+		(fields_autoplaced yes)
+		(effects
+			(font
+				(size 1.27 1.27)
+			)
+			(justify left bottom)
+		)
+	)
 	(label "Neutral"
-		(at 171.45 82.55 180)
+		(at 171.45 85.09 180)
 		(fields_autoplaced yes)
 		(effects
@@
 	)
 	(label "UART_TX"
-		(at 173.99 128.27 180)
+		(at 173.99 130.81 180)
 		(fields_autoplaced yes)
 		(effects
@@
 	)
 	(label "GearSelector"
-		(at 121.92 48.26 180)
+		(at 121.92 50.8 180)
 		(fields_autoplaced yes)
 		(effects
@@
 		)
 	)
+	(label "DRLLeftOut"
+		(at 264.16 111.76 0)
+		(fields_autoplaced yes)
+		(effects
+			(font
+				(size 1.27 1.27)
+			)
+			(justify left bottom)
+		)
+	)
 	(label "SupBattMonitor"
 		(at 154.94 158.75 180)
@@
 		)
 	)
+	(label "HazardIn"
+		(at 262.89 87.63 0)
+		(fields_autoplaced yes)
+		(effects
+			(font
+				(size 1.27 1.27)
+			)
+			(justify left bottom)
+		)
+	)
 	(label "DIExtra1"
 		(at 173.99 118.11 180)
@@
 		)
 	)
+	(label "Neutral"
+		(at 270.51 139.7 0)
+		(fields_autoplaced yes)
+		(effects
+			(font
+				(size 1.27 1.27)
+			)
+			(justify left bottom)
+		)
+	)
 	(label "RSignalLightButton"
 		(at 121.92 38.1 180)
@@
 	)
 	(label "Reverse"
-		(at 171.45 85.09 180)
+		(at 171.45 87.63 180)
 		(fields_autoplaced yes)
 		(effects
@@
 	)
 	(label "Drive"
-		(at 171.45 80.01 180)
+		(at 171.45 82.55 180)
 		(fields_autoplaced yes)
 		(effects
@@
 		)
 	)
-	(label "SupBattMonitor"
-		(at 262.89 87.63 0)
+	(label "Drive"
+		(at 270.51 137.16 0)
 		(fields_autoplaced yes)
 		(effects
@@
 		)
 	)
-	(label "HazardIn"
+	(label "AccelIn"
 		(at 200.66 134.62 0)
 		(fields_autoplaced yes)
@@
 	)
 	(label "SupBattery"
-		(at 171.45 87.63 180)
+		(at 171.45 80.01 180)
 		(fields_autoplaced yes)
 		(effects
@@
 		)
 	)
+	(label "DRLRightOut"
+		(at 264.16 124.46 0)
+		(fields_autoplaced yes)
+		(effects
+			(font
+				(size 1.27 1.27)
+			)
+			(justify left bottom)
+		)
+	)
 	(label "ThermalShutoff"
 		(at 173.99 125.73 180)
@@
 	)
 	(label "HazardButton"
-		(at 121.92 50.8 180)
+		(at 121.92 48.26 180)
 		(fields_autoplaced yes)
 		(effects
@@
 		)
 	)
-	(label "AccelIn"
-		(at 262.89 80.01 0)
+	(label "CAN_L"
+		(at 171.45 90.17 180)
 		(fields_autoplaced yes)
 		(effects
@@
 				(size 1.27 1.27)
 			)
-			(justify left bottom)
+			(justify right bottom)
 		)
 	)
-	(label "ThermalShutoff"
-		(at 198.12 62.23 0)
+	(label "UART_RX"
+		(at 200.66 152.4 0)
 		(fields_autoplaced yes)
 		(effects
@@
 		)
 	)
-	(label "UART_RX"
-		(at 200.66 152.4 0)
+	(label "Reverse"
+		(at 270.51 142.24 0)
 		(fields_autoplaced yes)
 		(effects
@@
 		)
 	)
-	(label "LSignalLightOut"
-		(at 198.12 41.91 0)
+	(label "RSignalLightIn"
+		(at 264.16 134.62 0)
 		(fields_autoplaced yes)
 		(effects
@@
 	)
 	(label "UART_RX"
-		(at 173.99 130.81 180)
+		(at 173.99 128.27 180)
 		(fields_autoplaced yes)
 		(effects
@@
 		)
 	)
-	(label "Neutral"
-		(at 200.66 124.46 0)
-		(fields_autoplaced yes)
-		(effects
-			(font
-				(size 1.27 1.27)
-			)
-			(justify left bottom)
-		)
-	)
 	(label "CAN_TX"
 		(at 135.89 44.45 0)
@@
 		)
 	)
-	(label "DIExtra2"
+	(label "SupBattMonitor"
 		(at 264.16 132.08 0)
 		(fields_autoplaced yes)
@@
 		)
 	)
-	(label "Drive"
-		(at 200.66 129.54 0)
-		(fields_autoplaced yes)
-		(effects
-			(font
-				(size 1.27 1.27)
-			)
-			(justify left bottom)
-		)
-	)
-	(label "BrakeLightOut"
-		(at 199.39 44.45 0)
-		(fields_autoplaced yes)
-		(effects
-			(font
-				(size 1.27 1.27)
-			)
-			(justify left bottom)
-		)
-	)
-	(label "DRLRightOut"
-		(at 200.66 139.7 0)
+	(label "CAN_H"
+		(at 171.45 92.71 180)
 		(fields_autoplaced yes)
 		(effects
@@
 				(size 1.27 1.27)
 			)
-			(justify left bottom)
+			(justify right bottom)
 		)
 	)
@@
 		)
 	)
-	(label "RSignalLightOut"
-		(at 262.89 41.91 0)
-		(fields_autoplaced yes)
-		(effects
-			(font
-				(size 1.27 1.27)
-			)
-			(justify left bottom)
-		)
-	)
 	(label "DRLLeftNeg"
 		(at 17.78 163.83 0)
@@
 		)
 	)
-	(label "DIExtra1"
-		(at 200.66 137.16 0)
+	(label "ThermalShutoff"
+		(at 198.12 147.32 0)
 		(fields_autoplaced yes)
 		(effects
@@
 		)
 	)
-	(label "DIExtra2"
-		(at 173.99 120.65 180)
+	(label "LSignalLightIn"
+		(at 200.66 137.16 0)
 		(fields_autoplaced yes)
 		(effects
@@
 				(size 1.27 1.27)
 			)
-			(justify right bottom)
+			(justify left bottom)
 		)
 	)
-	(label "LSignalLightIn"
-		(at 264.16 106.68 0)
+	(label "DIExtra2"
+		(at 173.99 120.65 180)
 		(fields_autoplaced yes)
 		(effects
@@
 				(size 1.27 1.27)
 			)
-			(justify left bottom)
+			(justify right bottom)
 		)
 	)
-	(label "RSignalLightOut"
-		(at 66.04 105.41 0)
+	(label "BrakeLightOut"
+		(at 264.16 106.68 0)
 		(fields_autoplaced yes)
 		(effects
@@
 		)
 	)
-	(label "DRLLeftOut"
-		(at 262.89 44.45 0)
+	(label "RSignalLightOut"
+		(at 66.04 105.41 0)
 		(fields_autoplaced yes)
 		(effects
@@
 	(symbol
 		(lib_id "power:VCC")
-		(at 264.16 69.85 270)
+		(at 273.05 69.85 270)
 		(unit 1)
 		(exclude_from_sim no)
@@
 		(fields_autoplaced yes)
 		(property "Reference" "#PWR026"
-			(at 260.35 69.85 0)
+			(at 269.24 69.85 0)
 			(effects
 				(font
@@
 		)
 		(property "Value" "VCC"
-			(at 267.97 69.8499 90)
+			(at 276.86 69.8499 90)
 			(effects
 				(font
@@
 		)
 		(property "Footprint" ""
-			(at 264.16 69.85 0)
+			(at 273.05 69.85 0)
 			(effects
 				(font
@@
 		)
 		(property "Datasheet" ""
-			(at 264.16 69.85 0)
+			(at 273.05 69.85 0)
 			(effects
 				(font
@@
 		)
 		(property "Description" "Power symbol creates a global label with name \"VCC\""
-			(at 264.16 69.85 0)
+			(at 273.05 69.85 0)
 			(effects
 				(font
@@
 					(unit 1)
 				)
+			)
+		)
+	)
+	(symbol
+		(lib_id "DriverControlsLib:0001.2511.TR")
+		(at 265.43 69.85 0)
+		(unit 1)
+		(exclude_from_sim no)
+		(in_bom yes)
+		(on_board yes)
+		(dnp no)
+		(fields_autoplaced yes)
+		(property "Reference" "F6"
+			(at 265.43 69.85 0)
+			(effects
+				(font
+					(size 1.27 1.27)
+				)
+			)
+		)
+		(property "Value" "~"
+			(at 265.43 69.85 0)
+			(effects
+				(font
+					(size 1.27 1.27)
+				)
+				(hide yes)
+			)
+		)
+		(property "Footprint" "DriverControlsLib:FUSE-TH_BD5.4-W22.5-P27.5-D0.8"
+			(at 265.43 69.85 0)
+			(effects
+				(font
+					(size 1.27 1.27)
+				)
+				(hide yes)
+			)
+		)
+		(property "Datasheet" "https://atta.szlcsc.com/upload/public/pdf/source/20210428/9A503759987094315AD78A099D34569F.pdf"
+			(at 265.43 69.85 0)
+			(effects
+				(font
+					(size 1.27 1.27)
+				)
+				(hide yes)
+			)
+		)
+		(property "Description" "Type:Ceramic Tube Fuse Current Rating:5A Voltage Rating  (AC):250V Voltage Rating (DC):150V Operating Temperature:-55°C~+125°C Operating Temperature:-55°C~+125°C Breaking Capacity:1.5kA"
+			(at 265.43 69.85 0)
+			(effects
+				(font
+					(size 1.27 1.27)
+				)
+				(hide yes)
+			)
+		)
+		(property "Manufacturer Part" "0001.2511.TR"
+			(at 265.43 69.85 0)
+			(effects
+				(font
+					(size 1.27 1.27)
+				)
+				(hide yes)
+			)
+		)
+		(property "Manufacturer" "SCHURTER"
+			(at 265.43 69.85 0)
+			(effects
+				(font
+					(size 1.27 1.27)
+				)
+				(hide yes)
+			)
+		)
+		(property "Supplier Part" "C1972726"
+			(at 265.43 69.85 0)
+			(effects
+				(font
+					(size 1.27 1.27)
+				)
+				(hide yes)
+			)
+		)
+		(property "Supplier" "LCSC"
+			(at 265.43 69.85 0)
+			(effects
+				(font
+					(size 1.27 1.27)
+				)
+				(hide yes)
+			)
+		)
+		(property "LCSC Part Name" "250V"
+			(at 265.43 69.85 0)
+			(effects
+				(font
+					(size 1.27 1.27)
+				)
+				(hide yes)
+			)
+		)
+		(pin "1"
+		)
+		(pin "2"
+		)
+		(instances
+			(project "DC"
+				(path "/7c560bbd-cfc0-42ab-b727-e631475cbcaa"
+					(reference "F6")
+					(unit 1)
+				)

Commit message: finished first draft of routing
Connections:
- net DIExtra1: now also U7.CN7_32 (PA4)
- net DIExtra2: now also U7.CN7_34 (PB0)
- net DOExtra1: now also U7.CN7_36 (PC1); no longer U7.CN10_29 (PB5)
- no-connect marks 36 -> 42
Changed lines of the file:
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@@
-		)
-	)
-	(label "DOExtra1"
-		(at 200.66 142.24 0)
-		(fields_autoplaced yes)
-		(effects
-			(font
-				(size 1.27 1.27)
-			)
-			(justify left bottom)
 		)
 	)
@@
 	)
 	(label "HazardIn"
-		(at 262.89 87.63 0)
+		(at 267.97 87.63 0)
 		(fields_autoplaced yes)
 		(effects
@@
 		)
 	)
+	(label "DOExtra1"
+		(at 266.7 85.09 0)
+		(fields_autoplaced yes)
+		(effects
+			(font
+				(size 1.27 1.27)
+			)
+			(justify left bottom)
+		)
+	)
 	(label "AccelPedal"
 		(at 101.6 119.38 0)
@@
 		)
 	)
+	(label "DIExtra1"
+		(at 275.59 80.01 180)
+		(fields_autoplaced yes)
+		(effects
+			(font
+				(size 1.27 1.27)
+			)
+			(justify right bottom)
+		)
+	)
 	(label "GearSelector"
 		(at 101.6 170.18 0)
@@
 		(fields_autoplaced yes)
 		(effects
+			(font
+				(size 1.27 1.27)
+			)
+			(justify right bottom)
+		)
+	)
+	(label "DIExtra2"
+		(at 275.59 82.55 180)
+		(fields_autoplaced yes)
+		(effects

Commit message: fixed labels
Connections:
- net RSignalLightButton: no longer U7.CN10_1 (PC9)
- no-connect marks 42 -> 43
Changed lines of the file:
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@@
-		)
-	)
-	(label "RSignalLightIn"
-		(at 199.39 106.68 0)
-		(fields_autoplaced yes)
-		(effects
-			(font
-				(size 1.27 1.27)
-			)
-			(justify left bottom)
 		)
 	)
